Commit message: Progress on URDF file

File: urdf/bumperbot.urdf.xacro (robot description, xacro)
@@ -14,5 +14,19 @@
         <parent link="base_footprint"/>
         <child link="base_link"/>
-        <origin rpy="0 0 0" xyz="0 0 0.33"/> <!-- While the base link is oriented the same as the base footprint and intersect the axis of the wheels of the robot. And so, as we can see from this 3D model of the robot, the base link is 33mm height. So as we saw these two links. So the base footprint and the base link are oriented the same. So we can set the channel to zero to indicate that there is no relative orientation among them. And also we saw that the base link is above the base footprint of 33mm. So let's set the X, Y, Z to zero zero and 0.0 33. We can save our model and now we can already visualize our robot model in order to see the two links that we have created and how they are connected to each other.-->
+        <origin rpy="0 0 0" xyz="0 0 0.033"/> <!-- While the base link is oriented the same as the base footprint and intersect the axis of the wheels of the robot. And so, as we can see from this 3D model of the robot, the base link is 33mm height. So as we saw these two links. So the base footprint and the base link are oriented the same. So we can set the channel to zero to indicate that there is no relative orientation among them. And also we saw that the base link is above the base footprint of 33mm. So let's set the X, Y, Z to zero zero and 0.0 33. We can save our model and now we can already visualize our robot model in order to see the two links that we have created and how they are connected to each other.-->
+    </joint>
+    <link name="wheel_right_link">
+        <visual> <!-- Mesh -->
+            <origin rpy="1.57 0 0" xyz="0 0 0"/>
+            <geometry>
+                <mesh filename="package://bumperbot_description/meshes/wheel_right_link.STL"/>
+            </geometry>
+        </visual>
+    </link>
+    <joint name="wheel_right_joint" type="continuous"> <!-- So the type of this connection is continuous. And this basically means that the wheel can rotate around parent link. So the two links that are connected by this joint can move with respect to each other. So they are continuous. So this joint connects to link the parent of this connection. -->
+        <parent link="base_link"/>
+        <child link="wheel_right_link"/>
+        <axis xyz="0 1 0"/> <!-- This means wheel right link can rotate around Y-axis of the base link-->
+        <origin rpy="0 0 0" xyz="0 -0.07 0"/> <!-- Wheel right link is translated by 7 cms along -ve y axis-->
     </joint>
 </robot>
